Commit message: air_1

File: src/main_bot/description/robot_core.xacro (robot description, xacro)
@@ -22,4 +22,7 @@
   <material name="dark_grey">
     <color rgba="0.2 0.2 0.2 1.0"/>
+  </material>
+  <material name="green">
+    <color rgba="0.0 0.8 0.0 1.0"/>
   </material>
   <material name="black">
@@ -116,5 +119,5 @@
         <box size="${chassis_length} ${chassis_width} ${chassis_height}"/>
       </geometry>
-      <material name="dark_grey"/>
+      <material name="green"/>
     </visual>
     <collision>
@@ -127,4 +130,7 @@
     </xacro:inertial_box>
   </link>
+  <gazebo reference="base_link">
+    <material>Gazebo/Green</material>
+  </gazebo>
   <!-- ─── Joints ─── -->
   <joint name="base_footprint_joint" type="fixed">
