Commit message: add IMU

File: src/main_bot/description/lidar.xacro (robot description, xacro)
@@ -26,5 +26,5 @@
     <parent link="base_link"/>
     <child  link="lidar_frame"/>
-    <origin xyz="0 0 ${chassis_height/2 + lidar_height/2}" rpy="0 0 0"/>
+    <origin xyz="0 0 ${chassis_height/2 + 0.03 + lidar_height/2}" rpy="0 0 0"/>
   </joint>
   <!-- ─── Gazebo sensor ─── -->

File: src/main_bot/description/robot.urdf.xacro (robot description, xacro)
@@ -4,3 +4,4 @@
     <xacro:include filename="ros2_control.xacro"/>
     <xacro:include filename="lidar.xacro"/>
+    <xacro:include filename="imu.xacro"/>
 </robot>
