Commit message: f-over

File: src/main_bot/description/cart.urdf.xacro (robot description, xacro)
@@ -11,11 +11,11 @@
   <xacro:include filename="inertial.xacro"/>
   <!-- ─── Properties — footprint matches the robot's own chassis ─── -->
-  <xacro:property name="cart_length"        value="1.188"/>
-  <xacro:property name="cart_width"         value="0.632"/>
-  <xacro:property name="cart_height"        value="0.4"/>
+  <xacro:property name="cart_length"        value="0.297"/>
+  <xacro:property name="cart_width"         value="0.158"/>
+  <xacro:property name="cart_height"        value="0.1"/>
   <xacro:property name="cart_mass"          value="3.0"/>
-  <xacro:property name="cart_ground_clearance" value="0.03"/>
-  <xacro:property name="cwheel_radius"      value="0.15"/>
-  <xacro:property name="cwheel_width"       value="0.08"/>
+  <xacro:property name="cart_ground_clearance" value="0.0075"/>
+  <xacro:property name="cwheel_radius"      value="0.0375"/>
+  <xacro:property name="cwheel_width"       value="0.02"/>
   <xacro:property name="cwheel_mass"        value="0.3"/>
   <xacro:property name="cart_z_offset"  value="${cart_ground_clearance + cart_height/2}"/>
@@ -61,25 +61,25 @@
   <link name="cart_hook">
     <visual>
-      <origin xyz="0.2 0 0" rpy="0 0 0"/>
+      <origin xyz="0.05 0 0" rpy="0 0 0"/>
       <geometry>
-        <box size="0.4 0.06 0.04"/>
+        <box size="0.1 0.015 0.01"/>
       </geometry>
       <material name="cart_grey"/>
     </visual>
     <visual>
-      <origin xyz="0.4 0 0.05" rpy="0 0 0"/>
+      <origin xyz="0.1 0 0.0125" rpy="0 0 0"/>
       <geometry>
-        <cylinder radius="0.02" length="0.1"/>
+        <cylinder radius="0.005" length="0.025"/>
       </geometry>
       <material name="cart_black"/>
     </visual>
     <collision>
-      <origin xyz="0.2 0 0" rpy="0 0 0"/>
+      <origin xyz="0.05 0 0" rpy="0 0 0"/>
       <geometry>
-        <box size="0.4 0.06 0.04"/>
+        <box size="0.1 0.015 0.01"/>
       </geometry>
     </collision>
-    <xacro:inertial_box mass="0.2" x="0.4" y="0.06" z="0.04">
-      <origin xyz="0.2 0 0" rpy="0 0 0"/>
+    <xacro:inertial_box mass="0.2" x="0.1" y="0.015" z="0.01">
+      <origin xyz="0.05 0 0" rpy="0 0 0"/>
     </xacro:inertial_box>
   </link>
@@ -87,5 +87,5 @@
     <parent link="cart_body"/>
     <child  link="cart_hook"/>
-    <origin xyz="${cart_length/2} 0 ${-cart_height/2 + 0.08}" rpy="0 0 0"/>
+    <origin xyz="${cart_length/2} 0 ${-cart_height/2 + 0.02}" rpy="0 0 0"/>
   </joint>
   <!-- ─── Wheel macro — passive caster (unactuated, rolls freely) ─── -->

File: src/main_bot/description/robot_core.xacro (robot description, xacro)
@@ -3,16 +3,14 @@
   <xacro:include filename="inertial.xacro"/>
   <!-- ─── Properties ─── -->
-  <!-- Body scale ×4 (visualization request — lidar/imu sizes untouched, see their .xacro files) -->
-  <xacro:property name="body_scale"       value="4.0"/>
-  <xacro:property name="chassis_mass"     value="6.0"/>
-  <xacro:property name="chassis_length"   value="${0.297 * body_scale}"/>
-  <xacro:property name="chassis_width"    value="${0.158 * body_scale}"/>
-  <xacro:property name="chassis_height"   value="${0.062 * body_scale}"/>
-  <xacro:property name="ground_clearance" value="${0.022 * body_scale}"/>
-  <xacro:property name="wheel_mass"       value="0.6"/>
-  <xacro:property name="wheel_radius"     value="${0.05 * body_scale}"/>
-  <xacro:property name="wheel_width"      value="${0.029 * body_scale}"/>
-  <xacro:property name="wheelbase"        value="${0.21 * body_scale}"/>
-  <xacro:property name="track_width"      value="${0.217 * body_scale}"/>
+  <xacro:property name="chassis_mass"     value="2.0"/>
+  <xacro:property name="chassis_length"   value="0.297"/>
+  <xacro:property name="chassis_width"    value="0.158"/>
+  <xacro:property name="chassis_height"   value="0.062"/>
+  <xacro:property name="ground_clearance" value="0.022"/>
+  <xacro:property name="wheel_mass"       value="0.15"/>
+  <xacro:property name="wheel_radius"     value="0.05"/>
+  <xacro:property name="wheel_width"      value="0.029"/>
+  <xacro:property name="wheelbase"        value="0.21"/>
+  <xacro:property name="track_width"      value="0.217"/>
   <xacro:property name="steering_limit"    value="0.52"/>
   <xacro:property name="steering_effort"   value="10.0"/>
@@ -57,6 +55,6 @@
     <!-- Ma sát bánh dẫn động — cần cao để tạo lực đẩy robot -->
     <gazebo reference="${name}_wheel">
-      <mu>2.5</mu>
-      <mu2>2.5</mu2>
+      <mu>1.5</mu>
+      <mu2>1.5</mu2>
       <kp>1e6</kp>
       <kd>1.0</kd>
@@ -107,6 +105,6 @@
     <!-- Ma sát bánh trước — đủ để giữ hướng, không quá cao -->
     <gazebo reference="front_${name}_wheel">
-      <mu>1.8</mu>
-      <mu2>1.2</mu2>
+      <mu>1.0</mu>
+      <mu2>0.5</mu2>
       <kp>1e6</kp>
       <kd>1.0</kd>
